Commit message: 2026-03-04; modified core URDF

File: description/robot_core.xacro (robot description, xacro)
@@ -1,4 +1,5 @@
 <?xml version="1.0"?>
 <robot xmlns:xacro="http://www.ros.org/wiki/xacro" >
+    <xacro:include filename="inertial_macros.xacro"/>
     <material name="white">
         <color rgba="1 1 1 1"/>
@@ -11,5 +12,5 @@
     </material>
     <material name="black">
-        <color rgba="0.1 0.1 0.1 1"/>
+        <color rgba="0 0 0 1"/>
     </material>
     <!-- Base Link -->
@@ -30,7 +31,16 @@
             <material name="white"/>
         </visual>
+        <collision>
+            <origin xyz="0.15 0 0.075"/>
+            <geometry>
+                <box size="0.3 0.3 0.15"/>
+            </geometry>
+        </collision>
+        <xacro:inertial_box mass="0.5" x="0.3" y="0.3" z="0.15">
+            <origin xyz="0.15 0 0.075" rpy="0 0 0"/>
+        </xacro:inertial_box>
     </link>
     <!-- Left Wheel Link -->
-    <joint name="Left_Wheel_joint" type="continuous">
+    <joint name="left_wheel_joint" type="continuous">
         <parent link="base_link"/>
         <child link="left_wheel"/>
@@ -45,7 +55,15 @@
             <material name="blue"/>
         </visual>
+        <collision>>
+            <geometry>
+                <cylinder radius="0.05" length="0.04"/>
+            </geometry>
+        </collision>
+        <xacro:inertial_cylinder mass="0.1" length="0.04" radius="0.05">
+            <origin xyz="0 0 0" rpy="0 0 0"/>
+        </xacro:inertial_cylinder>
     </link>
     <!-- Right Wheel Link -->
-    <joint name="Right_Wheel_joint" type="continuous">
+    <joint name="right_wheel_joint" type="continuous">
         <parent link="base_link"/>
         <child link="right_wheel"/>
@@ -60,18 +78,34 @@
             <material name="blue"/>
         </visual>
+        <collision>
+            <geometry>
+                <cylinder radius="0.05" length="0.04"/>
+            </geometry>
+        </collision>
+        <xacro:inertial_cylinder mass="0.1" length="0.04" radius="0.05">
+            <origin xyz="0 0 0" rpy="0 0 0"/>
+        </xacro:inertial_cylinder>
     </link>
     <!-- Caster Wheel Link -->
     <joint name="caster_wheel_joint" type="fixed">
-        <parent link="base_link"/>
+        <parent link="chassis"/>
         <child link="caster_wheel"/>
-        origin xyz="0.24 0 0"/>
+        <origin xyz="0.24 0 0"/>
     </joint>
-    <link name="caster_wheel">
-        <visual>
-            <geometry>
-                <sphere radius="0.03"/>sphere radius="0.05"/>
-            </geometry>
-            <material name="black"/>
-        </visual>
+        <link name="caster_wheel">
+            <visual>
+                <geometry>
+                    <sphere radius="0.05"/>
+                </geometry>
+                <material name="black"/>
+            </visual>
+            <collision>>
+                <geometry>
+                    <sphere radius="0.05"/>
+                </geometry>
+            </collision>
+            <xacro:inertial_sphere mass="0.1" radius="0.05">
+                <origin xyz="0 0 0" rpy="0 0 0"/>
+            </xacro:inertial_sphere>
     </link>
 </robot>

Commit message: 2026-03-04; Test gazebo control

File: description/robot_core.xacro (robot description, xacro)
@@ -47,4 +47,5 @@
         <origin xyz="0 0.175 0" rpy="-${pi/2} 0 0"/>
         <axis xyz="0 0 1"/>
+        <limit effort="0.05" velocity="10.0"/>
     </joint>
     <link name="left_wheel">
@@ -57,5 +58,5 @@
         <collision>>
             <geometry>
-                <cylinder radius="0.05" length="0.04"/>
+                <sphere radius="0.05" />
             </geometry>
         </collision>
@@ -70,4 +71,5 @@
         <origin xyz="0 -0.175 0" rpy="${pi/2} 0 0"/>
         <axis xyz="0 0 -1"/>
+        <limit effort="0.05" velocity="10.0"/>
     </joint>
     <link name="right_wheel">
@@ -80,5 +82,5 @@
         <collision>
             <geometry>
-                <cylinder radius="0.05" length="0.04"/>
+                <sphere radius="0.05" />
             </geometry>
         </collision>
@@ -93,19 +95,23 @@
         <origin xyz="0.24 0 0"/>
     </joint>
-        <link name="caster_wheel">
-            <visual>
-                <geometry>
-                    <sphere radius="0.05"/>
-                </geometry>
-                <material name="black"/>
-            </visual>
-            <collision>>
-                <geometry>
-                    <sphere radius="0.05"/>
-                </geometry>
-            </collision>
-            <xacro:inertial_sphere mass="0.1" radius="0.05">
-                <origin xyz="0 0 0" rpy="0 0 0"/>
-            </xacro:inertial_sphere>
+    <link name="caster_wheel">
+        <visual>
+            <geometry>
+                <sphere radius="0.05"/>
+            </geometry>
+            <material name="black"/>
+        </visual>
+        <collision>>
+            <geometry>
+                <sphere radius="0.05"/>
+            </geometry>
+        </collision>
+        <xacro:inertial_sphere mass="0.1" radius="0.05">
+            <origin xyz="0 0 0" rpy="0 0 0"/>
+        </xacro:inertial_sphere>
     </link>
+    <gazebo reference="caster_wheel">
+        <mu1 value="0.0"/>
+        <mu2 value="0.0"/>
+    </gazebo>
 </robot>

Commit message: 2026-03-06; add my_obstacle_world.sdf

File: description/robot_core.xacro (robot description, xacro)
@@ -14,5 +14,7 @@
         <color rgba="0 0 0 1"/>
     </material>
-    <!-- Base Link -->
+    <material name="red">
+        <color rgba="1 0 0 1"/>
+    </material>
     <link name="base_link">
     </link>

Commit message: 2026-03-18; SLAM with slam_toolbox

File: description/robot_core.xacro (robot description, xacro)
@@ -18,4 +18,12 @@
     </material>
     <link name="base_link">
+    </link>
+    <!-- BASE_FOOTPRINT -->
+    <joint name="base_footprint_joint" type="fixed">
+        <parent link="base_link"/>
+        <child link="base_footprint"/>
+        <origin xyz="0 0 0" rpy="0 0 0"/>
+    </joint>
+    <link name="base_footprint">
     </link>
     <!-- Chassis Link -->
